File: icescreamer.sch (KiCad schematic (older format))
At the start: 47 parts, among them CON1 BARREL_JACK, J1 JACK, J2 JACK, P1 CONN_2, Q1 NPN, Q2 NPN, SW1 3PDT, U1 TL072, U2 TLE2426NR

Commit message: Add new footprints
Parts:
- removed RV1: 500KA, ~, symbol POT
- removed RV2: 20K, ~, symbol POT
- removed RV3: 100KA, ~, symbol POT
- added RV1: 500KA, ~, symbol PASSIVES_POT_W_SHIELD
- added RV2: 20K, ~, symbol PASSIVES_POT_W_SHIELD
- added RV3: 100KA, ~, symbol PASSIVES_POT_W_SHIELD
Connections:
- wire segments 104 -> 109
Changed lines of the file:
@@
 Sheet 1 1
 Title "TubeScreamer"
-Date "7 apr 2015"
+Date "3 may 2015"
 Rev "0.1"
 Comp "DEF"
@@
 $EndComp
 $Comp
-L POT RV1
-U 1 1 55119907
-P 5400 3700
-F 0 "RV1" H 5400 3600 50  0000 C CNN
-F 1 "500KA" H 5400 3700 50  0000 C CNN
-F 2 "~" H 5400 3700 60  0000 C CNN
-F 3 "~" H 5400 3700 60  0000 C CNN
-	1    5400 3700
-	1    0    0    -1
-$EndComp
-$Comp
 L GND #PWR04
 U 1 1 55119BA9
@@
 $EndComp
 $Comp
-L POT RV2
-U 1 1 55119F6C
-P 7700 2000
-F 0 "RV2" H 7700 1900 50  0000 C CNN
-F 1 "20K" H 7700 2000 50  0000 C CNN
-F 2 "~" H 7700 2000 60  0000 C CNN
-F 3 "~" H 7700 2000 60  0000 C CNN
-	1    7700 2000
-	1    0    0    1
-$EndComp
-$Comp
 L R R10
 U 1 1 55119FCE
@@
 $EndComp
 $Comp
-L POT RV3
-U 1 1 55119FF1
-P 10550 2250
-F 0 "RV3" H 10550 2150 50  0000 C CNN
-F 1 "100KA" H 10550 2250 50  0000 C CNN
-F 2 "~" H 10550 2250 60  0000 C CNN
-F 3 "~" H 10550 2250 60  0000 C CNN
-	1    10550 2250
-	0    1    1    0
-$EndComp
-$Comp
 L -5V #PWR08
 U 1 1 5511AC60
@@
 Wire Notes Line
 	7350 4500 5500 4500
+$Comp
+L PASSIVES_POT_W_SHIELD RV1
+U 1 1 55464106
+P 5400 3700
+F 0 "RV1" H 5550 3600 50  0000 C CNN
+F 1 "500KA" H 5400 3700 50  0000 C CNN
+F 2 "~" H 5400 3700 60  0000 C CNN
+F 3 "~" H 5400 3700 60  0000 C CNN
+	1    5400 3700
+	1    0    0    -1
+$EndComp
+$Comp
+L PASSIVES_POT_W_SHIELD RV3
+U 1 1 55464122
+P 10550 2250
+F 0 "RV3" H 10700 2150 50  0000 C CNN
+F 1 "100KA" H 10550 2250 50  0000 C CNN
+F 2 "~" H 10550 2250 60  0000 C CNN
+F 3 "~" H 10550 2250 60  0000 C CNN
+	1    10550 2250
+	0    1    1    0
+$EndComp
+$Comp
+L PASSIVES_POT_W_SHIELD RV2
+U 1 1 55464137
+P 7700 2000
+F 0 "RV2" H 7850 1900 50  0000 C CNN
+F 1 "20K" H 7700 2000 50  0000 C CNN
+F 2 "~" H 7700 2000 60  0000 C CNN
+F 3 "~" H 7700 2000 60  0000 C CNN
+	1    7700 2000
+	-1   0    0    1
+$EndComp
+$Comp
+L GND #PWR032
+U 1 1 55464198
+P 5400 3950
+F 0 "#PWR032" H 5400 3950 30  0001 C CNN
+F 1 "GND" H 5400 3880 30  0001 C CNN
+F 2 "" H 5400 3950 60  0000 C CNN
+F 3 "" H 5400 3950 60  0000 C CNN
+	1    5400 3950
+	1    0    0    -1
+$EndComp
+Wire Wire Line
+	5400 3950 5400 3850
+$Comp
+L GND #PWR033
+U 1 1 5546419F
+P 10300 2350
+F 0 "#PWR033" H 10300 2350 30  0001 C CNN
+F 1 "GND" H 10300 2280 30  0001 C CNN
+F 2 "" H 10300 2350 60  0000 C CNN
+F 3 "" H 10300 2350 60  0000 C CNN
+	1    10300 2350
+	1    0    0    -1
+$EndComp
+Wire Wire Line
+	10300 2350 10300 2250
+Wire Wire Line
+	10300 2250 10400 2250
+$Comp
+L GND #PWR034
+U 1 1 55464249
+P 7950 1900
+F 0 "#PWR034" H 7950 1900 30  0001 C CNN
+F 1 "GND" H 7950 1830 30  0001 C CNN
+F 2 "" H 7950 1900 60  0000 C CNN
+F 3 "" H 7950 1900 60  0000 C CNN
+	1    7950 1900
+	1    0    0    -1
+$EndComp
+Wire Wire Line
+	7950 1850 7950 1900
+Wire Wire Line
+	7700 1850 7950 1850
 $EndSCHEMATC
