File: KiCad/icescreamer.kicad_pcb (KiCad board)
At the start: 2 copper layers, 48 x 98 mm, 47 parts, among them CON1 BARREL_JACK, J1 JACK, J2 JACK, P1 CONN_2, Q1 NPN, Q2 NPN, SW1 3PDT, U1 TL072, U2 TLE2426NR

Commit message: new edge cuts. It should work
Parts:
- removed C1: 0.02uF, C1-1
- removed C10, C14, C2, C9: 1uF, C1-1
- removed C11: 0.1Uf, C1
- removed C12, C13, C8: 0.1uF, C1
- removed C3: 0.047uF, C1-1
- removed C4: 51pF, C1-1
- removed C5, C6: 0.22uF, C1-1
- removed C7: 220uF, CP4
- removed CON1: BARREL_JACK, JACK_ALIM
- removed D1, D2, D4: DIODE, D3
- removed D3: LED, LED-5MM
- removed J1, J2: JACK, Conn_Jack_Female_635_THD
- removed P1: CONN_2, PIN_ARRAY_2X1
- removed Q1, Q2: NPN, TO92
- removed R1, R10, R12, R7: 1K, R3
- removed R11: 4K7, R3
- removed R13, R2: 510K, R3
- removed R14, R16, R3, R4, R8: 10K, R3
- removed R15: 100R, R3
- removed R17: 20K, R3
- removed R5: 4.7K, R3
- removed R6: 51K, R3
- removed R9: 220R, R3
- removed RV1: 500KA, Passives_BOURNS_PTV09A
- removed RV2: 20K, Passives_BOURNS_PTV09A
- removed RV3: 100KA, Passives_BOURNS_PTV09A
- removed SW1: 3PDT, Switches_Stomp_3PDT
- removed U1: TL072, DIP-8__300
- removed U2: TLE2426NR, DIP-8__300
Other:
- board size 48 x 98 mm -> 60 x 20 mm
