File: KiCad/icescreamer.kicad_pcb (KiCad board)
At the start: 2 copper layers, 60 x 85 mm, 85 parts, among them J1 Audio-Jack-3_3Switches, J2 Audio-Jack-3_3Switches, J3 Barrel_Jack_Switch, Q1 2SC1815, Q2 2SC1815, Q20 2SC1815, Q21 2SC1815, Q22 2SC1815, Q23 Q_NJFET_SGD, Q24 Q_NJFET_SGD, SW1 SW_TPDT, SW20 SW_Push, U1 NE5532

Commit message: V0.3 ready
Parts:
- added C14: C, Capacitor_SMD:C_0805_2012Metric_Pad1.15x1.40mm_HandSolder, F.Cu at (224.1, 66.7)
- added C15: C, Capacitor_SMD:C_0805_2012Metric_Pad1.15x1.40mm_HandSolder, F.Cu at (232.1, 66.8)
- added C16: C, Capacitor_SMD:C_0805_2012Metric_Pad1.15x1.40mm_HandSolder, F.Cu at (213.5, 74.2)
- added C17: C, Capacitor_SMD:C_0805_2012Metric_Pad1.15x1.40mm_HandSolder, F.Cu at (191.3, 64.6)
- added C18: C, Capacitor_SMD:C_0805_2012Metric_Pad1.15x1.40mm_HandSolder, F.Cu at (195.2, 76.9)
- added G***: LOGO, prueba:ice01, B.Cu at (213.8, 110.7)
- added G***: LOGO, prueba:ice00, B.Cu at (210.9, 110.8)
- added G***: LOGO, prueba:ice0, F.Cu at (230.8, 110.0)
- D4: footprint Connector_PinHeader_2.54mm:PinHeader_1x02_P2.54mm_Vertical -> Connector_PinHeader_2.00mm:PinHeader_1x02_P2.00mm_Vertical
- moved Q1 8.90 mm to (202.6, 89.9)
- moved Q23 8.89 mm to (191.1, 90.9)
- moved Q22 7.25 mm to (228.3, 125.3)
- moved R18 6.06 mm to (236.3, 126.6)
- moved R35 6.06 mm to (236.3, 124.3)
- moved R1 6.06 mm to (236.3, 131.1)
- moved R2 6.06 mm to (236.3, 128.8)
- moved JP1 3.24 mm to (228.0, 62.7)
- moved JP20 2.97 mm to (213.4, 113.2)
- moved JP21 2.87 mm to (213.4, 116.0)
- moved R4 2.67 mm to (195.1, 79.5)
- moved R3 2.60 mm to (195.1, 82.0), turned to 0 degrees
- moved C7 2.57 mm to (206.4, 70.2)
- moved C5 2.48 mm to (195.1, 84.4), turned to 180 degrees
- moved C3 2.41 mm to (213.6, 71.9)
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- renumbered SW20 to SW_TBP
Connections:
- J1 pad 5: (no net) -> Net-(J1-Pad5)
- J1 pad 6: (no net) -> Net-(J1-Pad6)
- J2 pad 4: (no net) -> Net-(J2-Pad4)
- J2 pad 5: (no net) -> Net-(J2-Pad5)
- J2 pad 6: (no net) -> Net-(J2-Pad6)
- POT1 pad 3: (no net) -> Net-(POT1-Pad3)
- SW1 pad 32: (no net) -> Net-(SW1-Pad32)
Routing:
- net GNDREF: track 252.1 -> 272.5 mm, vias 12 -> 14
- net Net-(R18-Pad2): track 23.1 -> 41.1 mm
- net LED_CATHODE: track 10.6 -> 27.4 mm, vias 0 -> 1
- net BATT-: track 30.1 -> 46.4 mm, vias 0 -> 2
- net JACK_IN: track 35.0 -> 50.6 mm
- net JACK_OUT: track 32.7 -> 18.3 mm, vias 2 -> 0
- net Net-(C20-Pad1): track 15.7 -> 29.9 mm, vias 0 -> 2
- net PSEUDO_OUT: track 57.3 -> 70.6 mm, vias 3 -> 1
- net EFF_IN: track 73.2 -> 84.8 mm
- net -VDC: track 27.2 -> 37.6 mm, vias 12 -> 16
- net PSEUDO_IN_2: track 35.5 -> 41.9 mm
- net PSEUDO_IN_1: track 21.3 -> 17.5 mm, vias 1 -> 0
- net Net-(D22-Pad2): track 73.9 -> 70.3 mm
- net Net-(D21-Pad2): track 64.1 -> 67.7 mm
- net Net-(D20-Pad2): track 59.5 -> 57.6 mm, vias 2 -> 1
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Other:
- board text added: "Board & upgrades: JorFru"
- board text added: "DC Power"
- board text added: "Input"
- board text added: "Output"
- board text added: "Short both for PSB"
- board text added: "Short for TruBy"
- board text added: "Status LED"
- board text added: "github.com/UC3Music/IceScreamer"

Commit message: V0.3 release
Parts:
- removed the G*** at (213.8, 110.7)
- added G***: LOGO, prueba:ice03, B.Cu at (213.8, 110.7)
- Q1, Q2, Q20, Q21, Q22: value 2SC1815 -> BC547; footprint drawdio:TO-92_SOT23_JorFru_compact -> IceScreamer:TO-92_SOT23_JorFru_compact
- SW1: value SW_TPDT -> SW_TruBy
- moved Q22 3.42 mm to (229.6, 128.5), turned to 90 degrees
- moved Q2 3.04 mm to (232.3, 90.4), turned to 0 degrees
- moved Q1 2.59 mm to (200.2, 90.9), turned to 0 degrees
- moved Q21 0.71 mm to (194.4, 124.7)
- moved Q20 0.63 mm to (195.6, 120.9)
- moved POT1 0.37 mm to (197.8, 58.4)
- renumbered SW_TBP to SW20
Connections:
- Q1 pad 1: PSEUDO_IN_1 -> +VDC
- Q1 pad 2: +VDC -> Net-(Q1-Pad2)
- Q1 pad 3: Net-(Q1-Pad3) -> PSEUDO_IN_1
- Q2 pad 1: Net-(Q2-Pad1) -> +VDC
- Q2 pad 2: +VDC -> Net-(C12-Pad1)
- Q2 pad 3: Net-(C12-Pad1) -> Net-(Q2-Pad3)
- Q20 pad 1: Net-(D22-Pad2) -> Net-(C23-Pad2)
- Q20 pad 2: Net-(C23-Pad2) -> Net-(C24-Pad2)
- Q20 pad 3: Net-(C24-Pad2) -> Net-(D22-Pad2)
- Q21 pad 1: Net-(D22-Pad2) -> Net-(C24-Pad1)
- Q21 pad 2: Net-(C24-Pad1) -> Net-(C23-Pad1)
- Q21 pad 3: Net-(C23-Pad1) -> Net-(D22-Pad2)
- Q22 pad 1: Net-(D22-Pad2) -> Net-(D23-Pad2)
- Q22 pad 2: Net-(D23-Pad2) -> Net-(Q22-Pad2)
- Q22 pad 3: Net-(Q22-Pad3) -> Net-(D22-Pad2)
- R15 pad 1: Net-(Q2-Pad1) -> Net-(Q2-Pad3)
- R16 pad 2: Net-(Q2-Pad1) -> Net-(Q2-Pad3)
- R3 pad 1: Net-(Q1-Pad3) -> Net-(Q1-Pad2)
- R33 pad 2: Net-(Q22-Pad3) -> Net-(Q22-Pad2)
- R4 pad 1: Net-(Q1-Pad3) -> Net-(Q1-Pad2)
Routing:
- net Net-(Q22-Pad3): track 65.0 -> 0.00 mm, vias 2 -> 0
- net Net-(Q22-Pad2): track 0.00 -> 64.5 mm, vias 0 -> 2
- net Net-(Q2-Pad3): track 0.00 -> 16.2 mm
- net Net-(Q1-Pad2): track 0.00 -> 15.5 mm
- net Net-(Q1-Pad3): track 14.5 -> 0.00 mm
- net Net-(Q2-Pad1): track 13.6 -> 0.00 mm, vias 2 -> 0
- net Net-(D22-Pad2): track 70.3 -> 75.7 mm
- net GNDREF: track 272.5 -> 275.8 mm
- net Net-(C12-Pad1): track 17.5 -> 20.8 mm
- net Net-(D23-Pad2): track 7.35 -> 10.6 mm
- net PSEUDO_IN_1: track 17.5 -> 19.6 mm
- net Net-(C24-Pad1): track 16.8 -> 15.4 mm
- net Net-(C23-Pad1): track 13.3 -> 14.6 mm
- net Net-(D20-Pad2): track 57.6 -> 58.8 mm
- net Net-(D21-Pad2): track 67.7 -> 66.7 mm
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Other:
- board text added: "+"
- board text added: "-"
- board text added: "9V Batt"
- board text added: "CREAM"
- board text added: "ICE"
- board text added: "MILK"
- board text added: "S"
- board text added: "SW_Pseudo"
- board text added: "Short both for Pseudo"
- board text removed: "Short both for PSB"
