File: KiCad/icescreamer.sch (KiCad schematic (older format))
At the start: 47 parts, among them CON1 PWR_IN, J1 JACK, J2 JACK, P1 BAT_T, Q1 NPN, Q2 NPN, SW1 3PDT, U1 TL072

Commit message: Updated components on schematic with newer ones. EdgeCuts on board already has the proper size. Added custom potentiometer footprint.
Parts:
- removed D1, D2: DIODE, Diodes_ThroughHole:Diode_DO-41_SOD81_Vertical_KathodeUp, symbol DIODE
- removed J1, J2: JACK, def-footprints:CONN_Jack_Female_6.35mm_THD, symbol CONNECTORS_JACK_FEMALE_STEREO_6_PINS
- removed RV1: 500KA, symbol PASSIVES_POT_W_SHIELD
- removed RV2: 20K, symbol PASSIVES_POT_W_SHIELD
- removed RV3: 100KA, symbol PASSIVES_POT_W_SHIELD
- added D1, D2: D, symbol D
- added J1, J2: JACK_FEMALE_STEREO_6_PINS, symbol JACK_FEMALE_STEREO_6_PINS
- added RV1, RV2, RV3: POT, symbol POT
Connections:
- wire segments 104 -> 100
Changed lines of the file:
@@
 LIBS:valves
 LIBS:kicad-library
+LIBS:icescreamer
 LIBS:icescreamer-cache
 EELAYER 25 0
@@
 $EndComp
 $Comp
-L DIODE D1
-U 1 1 5511983F
-P 5500 4200
-F 0 "D1" H 5300 4250 40  0000 C CNN
-F 1 "DIODE" H 5700 4100 40  0000 C CNN
-F 2 "Diodes_ThroughHole:Diode_DO-41_SOD81_Vertical_KathodeUp" H 5500 4200 60  0000 C CNN
-F 3 "~" H 5500 4200 60  0000 C CNN
-	1    5500 4200
-	1    0    0    -1
-$EndComp
-$Comp
-L DIODE D2
-U 1 1 55119856
-P 5500 4450
-F 0 "D2" H 5350 4500 40  0000 C CNN
-F 1 "DIODE" H 5700 4400 40  0000 C CNN
-F 2 "Diodes_ThroughHole:Diode_DO-41_SOD81_Vertical_KathodeUp" H 5500 4450 60  0000 C CNN
-F 3 "~" H 5500 4450 60  0000 C CNN
-	1    5500 4450
-	-1   0    0    1
-$EndComp
-$Comp
 L TL072 U1
 U 1 1 5511989A
@@
 $EndComp
 $Comp
-L -5V #PWR18
+L -5V #PWR16
 U 1 1 5511AC60
 P 8600 3750
-F 0 "#PWR18" H 8600 3890 20  0001 C CNN
+F 0 "#PWR16" H 8600 3890 20  0001 C CNN
 F 1 "-5V" H 8600 3860 30  0000 C CNN
 F 2 "" H 8600 3750 60  0000 C CNN
@@
 $EndComp
 $Comp
-L -5V #PWR13
+L -5V #PWR12
 U 1 1 5511AD56
 P 7750 4800
-F 0 "#PWR13" H 7750 4940 20  0001 C CNN
+F 0 "#PWR12" H 7750 4940 20  0001 C CNN
 F 1 "-5V" H 7750 4910 30  0000 C CNN
 F 2 "" H 7750 4800 60  0000 C CNN
@@
 $EndComp
 $Comp
-L -5V #PWR10
+L -5V #PWR9
 U 1 1 5511ADA3
 P 6900 3850
-F 0 "#PWR10" H 6900 3990 20  0001 C CNN
+F 0 "#PWR9" H 6900 3990 20  0001 C CNN
 F 1 "-5V" H 6900 3960 30  0000 C CNN
 F 2 "" H 6900 3850 60  0000 C CNN
@@
 $EndComp
 $Comp
-L -5V #PWR30
+L -5V #PWR25
 U 1 1 5511B635
 P 13700 4650
-F 0 "#PWR30" H 13700 4790 20  0001 C CNN
+F 0 "#PWR25" H 13700 4790 20  0001 C CNN
 F 1 "-5V" H 13700 4760 30  0000 C CNN
 F 2 "" H 13700 4650 60  0000 C CNN
@@
 $EndComp
 $Comp
-L -5V #PWR29
+L -5V #PWR24
 U 1 1 5511B63B
 P 12500 4650
-F 0 "#PWR29" H 12500 4790 20  0001 C CNN
+F 0 "#PWR24" H 12500 4790 20  0001 C CNN
 F 1 "-5V" H 12500 4760 30  0000 C CNN
 F 2 "" H 12500 4650 60  0000 C CNN
@@
 $EndComp
 $Comp
-L -5V #PWR23
+L -5V #PWR19
 U 1 1 5519D0B4
 P 9750 6800
-F 0 "#PWR23" H 9750 6940 20  0001 C CNN
+F 0 "#PWR19" H 9750 6940 20  0001 C CNN
 F 1 "-5V" H 9750 6910 30  0000 C CNN
 F 2 "" H 9750 6800 60  0000 C CNN
@@
 $EndComp
 $Comp
-L -5V #PWR24
+L -5V #PWR20
 U 1 1 5519D536
 P 9800 8200
-F 0 "#PWR24" H 9800 8340 20  0001 C CNN
+F 0 "#PWR20" H 9800 8340 20  0001 C CNN
 F 1 "-5V" H 9800 8310 30  0000 C CNN
 F 2 "" H 9800 8200 60  0000 C CNN
@@
 $EndComp
 $Comp
-L -5V #PWR12
+L -5V #PWR11
 U 1 1 5519D5AB
 P 7350 8300
-F 0 "#PWR12" H 7350 8440 20  0001 C CNN
+F 0 "#PWR11" H 7350 8440 20  0001 C CNN
 F 1 "-5V" H 7350 8410 30  0000 C CNN
 F 2 "" H 7350 8300 60  0000 C CNN
@@
 $EndComp
 $Comp
-L -5V #PWR15
+L -5V #PWR13
 U 1 1 5519E73F
 P 8000 8150
-F 0 "#PWR15" H 8000 8290 20  0001 C CNN
+F 0 "#PWR13" H 8000 8290 20  0001 C CNN
 F 1 "-5V" H 8000 8260 30  0000 C CNN
 F 2 "" H 8000 8150 60  0000 C CNN
@@
 	3800 4100 3800 4000
 Wire Wire Line
-	4400 3100 4950 3100
+	4400 3100 5150 3100
 Wire Wire Line
 	4600 3200 4600 3100
 Connection ~ 4600 3100
 Wire Wire Line
-	4950 3300 4900 3300
+	4900 3300 5150 3300
 Wire Wire Line
 	4900 3300 4900 4600
@@
 	6050 3200 6050 4850
 Wire Wire Line
-	4900 4200 5300 4200
+	4900 4200 5350 4200
 Connection ~ 4900 3950
 Wire Wire Line
-	4900 4450 5300 4450
+	4900 4450 5350 4450
 Connection ~ 4900 4200
 Wire Wire Line
-	6050 4200 5700 4200
+	5650 4200 6050 4200
 Connection ~ 6050 3950
 Connection ~ 6050 4200
 Connection ~ 4900 4450
 Wire Wire Line
-	4900 5100 5200 5100
+	4900 5100 5300 5100
 Wire Wire Line
 	5450 4950 5450 4850
@@
 	4600 5100 4600 5150
 Wire Wire Line
-	5350 3650 5350 3600
-Wire Wire Line
-	5350 2800 5350 2750
+	5350 3500 5350 3650
+Wire Wire Line
+	5350 2750 5350 2900
 Wire Wire Line
 	6700 3200 8200 3200
@@
 	8850 4200 9250 4200
 Wire Wire Line
-	8000 3400 8200 3400
-Wire Wire Line
-	9200 3300 9400 3300
+	7900 3400 8400 3400
+Wire Wire Line
+	9000 3300 9400 3300
 Wire Wire Line
 	9250 4200 9250 3300
@@
 	10750 3650 11450 3650
 Wire Wire Line
-	7500 3400 7450 3400
+	7450 3400 7600 3400
 Wire Wire Line
 	7450 3400 7450 3200
@@
 	8100 3400 8100 4200
 Wire Wire Line
-	8600 3750 8600 3700
+	8600 3600 8600 3750
 Wire Wire Line
 	7200 3900 7200 3800
@@
 	5950 3200 6200 3200
 Wire Wire Line
-	10600 3900 10600 4150
+	10600 3800 10600 4150
 Wire Wire Line
 	11850 3650 12200 3650
@@
 	12000 4350 12000 4300
 Wire Wire Line
-	10600 3400 10600 3300
+	10600 3300 10600 3500
 Wire Wire Line
 	6300 6750 6500 6750
@@
 Wire Wire Line
 	7050 6200 6300 6200
-NoConn ~ 5700 5100
-Wire Wire Line
-	5700 4450 6050 4450
+Wire Wire Line
+	5650 4450 6050 4450
 $Comp
 L +5V #PWR010
@@
 $EndComp
 Wire Wire Line
-	8600 2850 8600 2900
+	8600 2850 8600 3000
 $Comp
 L +5V #PWR012
@@
 Wire Notes Line
 	11350 3900 10700 3900
-$Comp
-L CONNECTORS_JACK_FEMALE_STEREO_6_PINS J1
-U 1 1 5524220A
-P 6400 7800
-F 0 "J1" H 5800 7350 60  0000 C CNN
-F 1 "JACK" H 5900 8100 60  0000 C CNN
-F 2 "def-footprints:CONN_Jack_Female_6.35mm_THD" H 6850 7750 60  0000 C CNN
-F 3 "~" H 6850 7750 60  0000 C CNN
-	1    6400 7800
-	1    0    0    -1
-$EndComp
 Text Notes 5450 8100 2    60   ~ 0
 INPUT
@@
 	6950 8050 7350 8050
 Connection ~ 7350 8050
-$Comp
-L CONNECTORS_JACK_FEMALE_STEREO_6_PINS J2
-U 1 1 55242A87
-P 10500 7850
-F 0 "J2" H 9900 7400 60  0000 C CNN
-F 1 "JACK" H 10000 8150 60  0000 C CNN
-F 2 "def-footprints:CONN_Jack_Female_6.35mm_THD" H 10950 7800 60  0000 C CNN
-F 3 "~" H 10950 7800 60  0000 C CNN
-	1    10500 7850
-	-1   0    0    -1
-$EndComp
 NoConn ~ 9950 8200
 NoConn ~ 9950 7800
@@
 Wire Notes Line
 	7400 5900 5550 5900
-$Comp
-L PASSIVES_POT_W_SHIELD RV1
-U 1 1 55464106
-P 5450 5100
-F 0 "RV1" H 5600 5000 50  0000 C CNN
-F 1 "500KA" H 5450 5100 50  0000 C CNN
-F 2 "" H 5450 5100 60  0000 C CNN
-F 3 "~" H 5450 5100 60  0000 C CNN
-	1    5450 5100
-	1    0    0    -1
-$EndComp
-$Comp
-L PASSIVES_POT_W_SHIELD RV3
-U 1 1 55464122
-P 10600 3650
-F 0 "RV3" H 10750 3550 50  0000 C CNN
-F 1 "100KA" H 10600 3650 50  0000 C CNN
-F 2 "" H 10600 3650 60  0000 C CNN
-F 3 "~" H 10600 3650 60  0000 C CNN
-	1    10600 3650
-	0    1    1    0
-$EndComp
-$Comp
-L PASSIVES_POT_W_SHIELD RV2
-U 1 1 55464137
-P 7750 3400
-F 0 "RV2" H 7900 3300 50  0000 C CNN
-F 1 "20K" H 7750 3400 50  0000 C CNN
-F 2 "" H 7750 3400 60  0000 C CNN
-F 3 "~" H 7750 3400 60  0000 C CNN
-	1    7750 3400
-	-1   0    0    1
-$EndComp
-$Comp
-L GND-RESCUE-icescreamer #PWR014
-U 1 1 55464198
-P 5450 5350
-F 0 "#PWR014" H 5450 5350 30  0001 C CNN
-F 1 "GND" H 5450 5280 30  0001 C CNN
-F 2 "" H 5450 5350 60  0000 C CNN
-F 3 "" H 5450 5350 60  0000 C CNN
-	1    5450 5350
-	1    0    0    -1
-$EndComp
-Wire Wire Line
-	5450 5350 5450 5250
-$Comp
-L GND-RESCUE-icescreamer #PWR015
-U 1 1 5546419F
-P 10350 3750
-F 0 "#PWR015" H 10350 3750 30  0001 C CNN
-F 1 "GND" H 10350 3680 30  0001 C CNN
-F 2 "" H 10350 3750 60  0000 C CNN
-F 3 "" H 10350 3750 60  0000 C CNN
-	1    10350 3750
-	1    0    0    -1
-$EndComp
-Wire Wire Line
-	10350 3750 10350 3650
-Wire Wire Line
-	10350 3650 10450 3650
-$Comp
-L GND-RESCUE-icescreamer #PWR016
-U 1 1 55464249
-P 8000 3300
-F 0 "#PWR016" H 8000 3300 30  0001 C CNN
-F 1 "GND" H 8000 3230 30  0001 C CNN
-F 2 "" H 8000 3300 60  0000 C CNN
-F 3 "" H 8000 3300 60  0000 C CNN
-	1    8000 3300
-	1    0    0    -1
-$EndComp
-Wire Wire Line
-	8000 3250 8000 3300
-Wire Wire Line
-	7750 3250 8000 3250
 $Comp
 L CAPAPOL C12
@@
 Connection ~ 10600 6800
 $Comp
-L PWR_FLAG #FLG017
+L PWR_FLAG #FLG014
 U 1 1 57FC5653
 P 9750 6300
-F 0 "#FLG017" H 9750 6395 50  0001 C CNN
+F 0 "#FLG014" H 9750 6395 50  0001 C CNN
 F 1 "PWR_FLAG" H 9750 6480 50  0000 C CNN
 F 2 "" H 9750 6300 60  0000 C CNN
@@
 $EndComp
 $Comp
-L PWR_FLAG #FLG018
+L PWR_FLAG #FLG015
 U 1 1 57FC8770
 P 10900 5800
-F 0 "#FLG018" H 10900 5895 50  0001 C CNN
+F 0 "#FLG015" H 10900 5895 50  0001 C CNN
 F 1 "PWR_FLAG" H 10900 5980 50  0000 C CNN
 F 2 "" H 10900 5800 60  0000 C CNN
@@
 $EndComp
 $Comp
-L PWR_FLAG #FLG019
+L PWR_FLAG #FLG016
 U 1 1 57FCA469
 P 10900 6800
-F 0 "#FLG019" H 10900 6895 50  0001 C CNN
+F 0 "#FLG016" H 10900 6895 50  0001 C CNN
 F 1 "PWR_FLAG" H 10900 6980 50  0000 C CNN
 F 2 "" H 10900 6800 60  0000 C CNN
@@
 	-1   0    0    1
 $EndComp
+Wire Wire Line
+	5750 3200 8400 3200
+$Comp
+L POT RV2
+U 1 1 596CF52B
+P 7750 3400
+F 0 "RV2" H 7750 3320 50  0000 C CNN
+F 1 "POT" H 7750 3400 50  0000 C CNN
+F 2 "" H 7750 3400 50  0000 C CNN
+F 3 "" H 7750 3400 50  0000 C CNN
+	1    7750 3400
+	-1   0    0    1
+$EndComp
+$Comp
+L POT RV1
+U 1 1 596CFA97
+P 5450 5100
+F 0 "RV1" H 5450 5020 50  0000 C CNN
+F 1 "POT" H 5450 5100 50  0000 C CNN
+F 2 "" H 5450 5100 50  0000 C CNN
+F 3 "" H 5450 5100 50  0000 C CNN
+	1    5450 5100
+	0    -1   -1   0
+$EndComp
+NoConn ~ 5450 5250
+$Comp
+L D D1
+U 1 1 596CFF85
+P 5500 4200
+F 0 "D1" H 5500 4300 50  0000 C CNN
+F 1 "D" H 5500 4100 50  0000 C CNN
+F 2 "" H 5500 4200 50  0000 C CNN
+F 3 "" H 5500 4200 50  0000 C CNN
+	1    5500 4200
+	1    0    0    -1
+$EndComp
+$Comp
+L D D2
+U 1 1 596CFFFA
+P 5500 4450
+F 0 "D2" H 5500 4550 50  0000 C CNN
+F 1 "D" H 5500 4350 50  0000 C CNN
+F 2 "" H 5500 4450 50  0000 C CNN
+F 3 "" H 5500 4450 50  0000 C CNN
+	1    5500 4450
+	1    0    0    -1
+$EndComp
+$Comp
+L POT RV3
+U 1 1 596D05A7
+P 10600 3650
+F 0 "RV3" H 10600 3570 50  0000 C CNN
+F 1 "POT" H 10600 3650 50  0000 C CNN
+F 2 "" H 10600 3650 50  0000 C CNN
+F 3 "" H 10600 3650 50  0000 C CNN
+	1    10600 3650
+	0    1    1    0
+$EndComp
+$Comp
+L JACK_FEMALE_STEREO_6_PINS J1
+U 1 1 596D6FF3
+P 6400 7800
+F 0 "J1" H 6950 7300 60  0000 C CNN
+F 1 "JACK_FEMALE_STEREO_6_PINS" H 5850 7300 60  0000 C CNN
+F 2 "" H 6850 7750 60  0000 C CNN
+F 3 "" H 6850 7750 60  0000 C CNN
+	1    6400 7800
+	1    0    0    -1
+$EndComp
+$Comp
+L JACK_FEMALE_STEREO_6_PINS J2
+U 1 1 596D8E31
+P 10500 7850
+F 0 "J2" H 11050 7350 60  0000 C CNN
+F 1 "JACK_FEMALE_STEREO_6_PINS" H 9950 7350 60  0000 C CNN
+F 2 "" H 10950 7800 60  0000 C CNN
+F 3 "" H 10950 7800 60  0000 C CNN
+	1    10500 7850
+	-1   0    0    -1
+$EndComp
 $EndSCHEMATC

Commit message: REDOed Schematic. Now supports both TrueBypass and PseudoBypass at the same time
Parts:
- removed C1: 0.02uF, Discret:C1-1, symbol C-RESCUE-icescreamer
- removed C10, C9: 0.1uF, Discret:C1-1, symbol C-RESCUE-icescreamer
- removed C11, C12: 220uF, Capacitors_ThroughHole:C_Radial_D5_L6_P2.5, symbol CAPAPOL
- removed C14, C2, C7: 1uF, Discret:C1-1, symbol C-RESCUE-icescreamer
- removed C3: 0.047uF, Discret:C1-1, symbol C-RESCUE-icescreamer
- removed C4: 51pF, Discret:C1-1, symbol C-RESCUE-icescreamer
- removed C5, C6: 0.22uF, Discret:C1-1, symbol C-RESCUE-icescreamer
- removed C8: 0.1Uf, Discret:C1-1, symbol C-RESCUE-icescreamer
- removed CON1: PWR_IN, symbol BARREL_JACK
- removed D3: LED, LEDs:LED-5MM, symbol LED
- removed D4: DIODE, Diodes_ThroughHole:Diode_P600_Vertical_AnodeUp, symbol DIODE
- removed J1, J2: JACK_FEMALE_STEREO_6_PINS, symbol JACK_FEMALE_STEREO_6_PINS
- removed P1: BAT_T, Connect:BARREL_JACK, symbol CONN_2
- removed Q1, Q2: NPN, symbol NPN
- removed R1, R10, R11, R7: 1K, symbol R-RESCUE-icescreamer
- removed R12: 20K, symbol R-RESCUE-icescreamer
- removed R13, R2: 510K, symbol R-RESCUE-icescreamer
- removed R14, R16, R17, R18, R3, R4, R8: 10K, symbol R-RESCUE-icescreamer
- removed R15: 100R, symbol R-RESCUE-icescreamer
- removed R19: 4K7, symbol R-RESCUE-icescreamer
- removed R5: 4.7K, symbol R-RESCUE-icescreamer
- removed R6: 51K, symbol R-RESCUE-icescreamer
- removed R9: 220R, symbol R-RESCUE-icescreamer
- removed RV1, RV2, RV3: POT, symbol POT
- removed SW1: 3PDT, symbol 3PDT
- removed U1: TL072, symbol TL072
- added BT1: Battery_Cell, Wire_Pads:SolderWirePad_2x_1-2mmDrill, symbol Battery_Cell
- added C1, C2: CP, Capacitors_THT:CP_Radial_D6.3mm_P2.50mm, symbol CP
- added C10, C11, C12, C13, C20, C21, C22, C23, C24, C25, C26, C27, C5, C6, C7, C8, C9: C, symbol C
- added C3, C4: C, Capacitors_THT:C_Rect_L7.0mm_W3.5mm_P2.50mm_P5.00mm, symbol C
- added D20, D21, D22, D3: D, symbol D
- added D23: D_Zener, symbol D_Zener
- added D4: LED, symbol LED
- added J1, J2: Audio-Jack-3_3Switches, footprints:IceJACK, symbol Audio-Jack-3_3Switches
- added JP1: TB, symbol Jumper
- added JP20, JP21: PSEUDO, symbol Jumper
- added POT1, POT2, POT3: POT, footprints:IcePOT, symbol POT
- added Q1, Q2, Q20, Q21, Q22: 2SC1815, TO_SOT_Packages_THT:TO-92_Molded_Narrow, symbol 2SC1815
- added Q23, Q24: Q_NJFET_SGD, symbol Q_NJFET_SGD
- added R1, R10, R11, R12, R13, R14, R15, R16, R17, R18, R19, R2, R20, R21, R22, R23, R24, R25, R26, R27, R28, R29, R3, R30, R31, R32, R33, R34, R35, R36, R4, R5, R6, R7, R8, R9: R, symbol R
- added SW1: SW_TPDT, symbol SW_TPDT
- added SW20: SW_Push, symbol SW_Push
- added U1: NE5532, symbol NE5532
Connections:
- net labels added: +VDC, -VDC, BATT-, EFF_IN, EFF_OUT, GNDREF, JACK_IN, JACK_OUT, LED_ANODE, LED_CATHODE, PSEUDO_IN_1, PSEUDO_IN_2, PSEUDO_OUT
- net labels removed: +5V, -5V, FX in, FX out, GND
- wire segments 100 -> 142
- no-connect marks 9 -> 7
Other:
- note removed: "INPUT"
- note removed: "OUTPUT JACK"
- note removed: "Optional: to convert\nlinear pot to log pot"
- note removed: "POWER INPUT"
- note removed: "Recommended transistors:\n(low noise)\nMPSA18\n2N5089"

Commit message: Asociadas las huellas a los componentes
Falta trabajar sobre esto, cotejando los componentes que se compraron y comprobar que las huellas que se eligen sean adecuadas para soldar a mano.
Parts:
- D2, D20, D21, D22, D23, D3: footprint (none) -> Diodes_SMD:D_SOD-323_HandSoldering
- D4: footprint (none) -> Pin_Headers:Pin_Header_Straight_1x02_Pitch2.54mm
- Q1, Q2, Q20, Q21, Q22: footprint TO_SOT_Packages_THT:TO-92_Molded_Narrow -> TO_SOT_Packages_SMD:SOT-323_SC-70_Handsoldering
- Q23, Q24: footprint (none) -> TO_SOT_Packages_SMD:SOT-323_SC-70_Handsoldering
- R1, R10, R11, R12, R13, R14, R15, R16, R17, R18, R19, R2, R20, R21, R22, R23, R24, R25, R26, R27, R28, R29, R3, R30, R31, R32, R33, R34, R35, R36, R4, R5, R6, R7, R8, R9: footprint (none) -> Resistors_SMD:R_0805_HandSoldering

Commit message: Updated asociación de huellas
Parts:
- C10, C11, C12, C13, C20, C21, C22, C23, C24, C25, C26, C27, C5, C6, C7, C8, C9, D1: footprint (none) -> Capacitors_SMD:C_0805_HandSoldering
- SW1: footprint (none) -> def-footprints:Switches_Stomp_Switch_3PDT
- SW20: footprint (none) -> def-footprints:Switches_Push_Switch_THD
Changed lines of the file:
@@
 F 0 "C5" H 2425 2300 50  0000 L CNN
 F 1 "C" H 2425 2100 50  0000 L CNN
-F 2 "" H 2438 2050 50  0001 C CNN
+F 2 "Capacitors_SMD:C_0805_HandSoldering" H 2438 2050 50  0001 C CNN
 F 3 "" H 2400 2200 50  0001 C CNN
 	1    2400 2200
@@
 F 0 "C6" H 4175 2500 50  0000 L CNN
 F 1 "C" H 4175 2300 50  0000 L CNN
-F 2 "" H 4188 2250 50  0001 C CNN
+F 2 "Capacitors_SMD:C_0805_HandSoldering" H 4188 2250 50  0001 C CNN
 F 3 "" H 4150 2400 50  0001 C CNN
 	1    4150 2400
@@
 F 0 "C7" H 4775 1900 50  0000 L CNN
 F 1 "C" H 4775 1700 50  0000 L CNN
-F 2 "" H 4788 1650 50  0001 C CNN
+F 2 "Capacitors_SMD:C_0805_HandSoldering" H 4788 1650 50  0001 C CNN
 F 3 "" H 4750 1800 50  0001 C CNN
 	1    4750 1800
@@
 F 0 "C8" H 4275 1250 50  0000 L CNN
 F 1 "C" H 4275 1050 50  0000 L CNN
-F 2 "" H 4288 1000 50  0001 C CNN
+F 2 "Capacitors_SMD:C_0805_HandSoldering" H 4288 1000 50  0001 C CNN
 F 3 "" H 4250 1150 50  0001 C CNN
 	1    4250 1150
@@
 F 0 "C9" H 6125 2650 50  0000 L CNN
 F 1 "C" H 6125 2450 50  0000 L CNN
-F 2 "" H 6138 2400 50  0001 C CNN
+F 2 "Capacitors_SMD:C_0805_HandSoldering" H 6138 2400 50  0001 C CNN
 F 3 "" H 6100 2550 50  0001 C CNN
 	1    6100 2550
@@
 F 0 "C10" H 6775 3300 50  0000 L CNN
 F 1 "C" H 6775 3100 50  0000 L CNN
-F 2 "" H 6788 3050 50  0001 C CNN
+F 2 "Capacitors_SMD:C_0805_HandSoldering" H 6788 3050 50  0001 C CNN
 F 3 "" H 6750 3200 50  0001 C CNN
 	1    6750 3200
@@
 F 0 "C11" H 7525 2500 50  0000 L CNN
 F 1 "C" H 7525 2300 50  0000 L CNN
-F 2 "" H 7538 2250 50  0001 C CNN
+F 2 "Capacitors_SMD:C_0805_HandSoldering" H 7538 2250 50  0001 C CNN
 F 3 "" H 7500 2400 50  0001 C CNN
 	1    7500 2400
@@
 F 0 "C12" H 9025 2750 50  0000 L CNN
 F 1 "C" H 9025 2550 50  0000 L CNN
-F 2 "" H 9038 2500 50  0001 C CNN
+F 2 "Capacitors_SMD:C_0805_HandSoldering" H 9038 2500 50  0001 C CNN
 F 3 "" H 9000 2650 50  0001 C CNN
 	1    9000 2650
@@
 F 0 "SW20" H 1150 6700 50  0000 L CNN
 F 1 "SW_Push" H 1100 6540 50  0000 C CNN
-F 2 "" H 1100 6800 50  0001 C CNN
+F 2 "def-footprints:Switches_Push_Switch_THD" H 1100 6800 50  0001 C CNN
 F 3 "" H 1100 6800 50  0001 C CNN
 	1    1100 6600
@@
 F 0 "C21" H 2075 4700 50  0000 L CNN
 F 1 "C" H 2075 4500 50  0000 L CNN
-F 2 "" H 2088 4450 50  0001 C CNN
+F 2 "Capacitors_SMD:C_0805_HandSoldering" H 2088 4450 50  0001 C CNN
 F 3 "" H 2050 4600 50  0001 C CNN
 	1    2050 4600
@@
 F 0 "C24" H 3925 5300 50  0000 L CNN
 F 1 "C" H 3925 5100 50  0000 L CNN
-F 2 "" H 3938 5050 50  0001 C CNN
+F 2 "Capacitors_SMD:C_0805_HandSoldering" H 3938 5050 50  0001 C CNN
 F 3 "" H 3900 5200 50  0001 C CNN
 	1    3900 5200
@@
 F 0 "C25" H 3275 5800 50  0000 L CNN
 F 1 "C" H 3275 5600 50  0000 L CNN
-F 2 "" H 3288 5550 50  0001 C CNN
+F 2 "Capacitors_SMD:C_0805_HandSoldering" H 3288 5550 50  0001 C CNN
 F 3 "" H 3250 5700 50  0001 C CNN
 	1    3250 5700
@@
 F 0 "C26" H 3625 5800 50  0000 L CNN
 F 1 "C" H 3625 5600 50  0000 L CNN
-F 2 "" H 3638 5550 50  0001 C CNN
+F 2 "Capacitors_SMD:C_0805_HandSoldering" H 3638 5550 50  0001 C CNN
 F 3 "" H 3600 5700 50  0001 C CNN
 	1    3600 5700
@@
 F 0 "C23" H 2975 5300 50  0000 L CNN
 F 1 "C" H 2975 5100 50  0000 L CNN
-F 2 "" H 2988 5050 50  0001 C CNN
+F 2 "Capacitors_SMD:C_0805_HandSoldering" H 2988 5050 50  0001 C CNN
 F 3 "" H 2950 5200 50  0001 C CNN
 	1    2950 5200
@@
 F 0 "C27" H 5025 4700 50  0000 L CNN
 F 1 "C" H 5025 4500 50  0000 L CNN
-F 2 "" H 5038 4450 50  0001 C CNN
+F 2 "Capacitors_SMD:C_0805_HandSoldering" H 5038 4450 50  0001 C CNN
 F 3 "" H 5000 4600 50  0001 C CNN
 	1    5000 4600
@@
 F 0 "C22" H 1775 6600 50  0000 L CNN
 F 1 "C" H 1775 6400 50  0000 L CNN
-F 2 "" H 1788 6350 50  0001 C CNN
+F 2 "Capacitors_SMD:C_0805_HandSoldering" H 1788 6350 50  0001 C CNN
 F 3 "" H 1750 6500 50  0001 C CNN
 	1    1750 6500
@@
 F 0 "C20" H 1675 3850 50  0000 L CNN
 F 1 "C" H 1675 3650 50  0000 L CNN
-F 2 "" H 1688 3600 50  0001 C CNN
+F 2 "Capacitors_SMD:C_0805_HandSoldering" H 1688 3600 50  0001 C CNN
 F 3 "" H 1650 3750 50  0001 C CNN
 	1    1650 3750
@@
 F 0 "D1" H 1400 1200 50  0000 C CNN
 F 1 "D" H 1400 1000 50  0000 C CNN
-F 2 "" H 1400 1100 50  0001 C CNN
+F 2 "Capacitors_SMD:C_0805_HandSoldering" H 1400 1100 50  0001 C CNN
 F 3 "" H 1400 1100 50  0001 C CNN
 	1    1400 1100
@@
 F 0 "SW1" H 7025 4400 50  0000 C CNN
 F 1 "SW_TPDT" H 7500 4400 50  0000 C CNN
-F 2 "" H 7200 4200 50  0001 C CNN
+F 2 "def-footprints:Switches_Stomp_Switch_3PDT" H 7200 4200 50  0001 C CNN
 F 3 "" H 7200 4200 50  0001 C CNN
 	1    7200 4200
@@
 F 0 "C13" H 10275 2950 50  0000 L CNN
 F 1 "C" H 10275 2750 50  0000 L CNN
-F 2 "" H 10288 2700 50  0001 C CNN
+F 2 "Capacitors_SMD:C_0805_HandSoldering" H 10288 2700 50  0001 C CNN
 F 3 "" H 10250 2850 50  0001 C CNN
 	1    10250 2850

Commit message: Lo mismo que antes pero un poco más afinado.
Parts:
- C10, C5, C7, C8: footprint Capacitors_SMD:C_0805_HandSoldering -> drawdio:Resistor_SMD+THT
- JP1, JP20, JP21: footprint (none) -> def-footprints:Miscellaneous_Solder_Jumper
- Q1, Q2: footprint TO_SOT_Packages_SMD:SOT-323_SC-70_Handsoldering -> drawdio:TO-92_SOT23_JorFru_compact
- SW1: footprint def-footprints:Switches_Stomp_Switch_3PDT -> Wire_Pads:SolderWirePad_2x_1-5mmDrill
Changed lines of the file:
@@
 F 0 "C5" H 2425 2300 50  0000 L CNN
 F 1 "C" H 2425 2100 50  0000 L CNN
-F 2 "Capacitors_SMD:C_0805_HandSoldering" H 2438 2050 50  0001 C CNN
+F 2 "drawdio:Resistor_SMD+THT" H 2438 2050 50  0001 C CNN
 F 3 "" H 2400 2200 50  0001 C CNN
 	1    2400 2200
@@
 F 0 "Q1" H 3750 2275 50  0000 L CNN
 F 1 "2SC1815" H 3750 2200 50  0000 L CNN
-F 2 "TO_SOT_Packages_SMD:SOT-323_SC-70_Handsoldering" H 3750 2125 50  0001 L CIN
+F 2 "drawdio:TO-92_SOT23_JorFru_compact" H 3750 2125 50  0001 L CIN
 F 3 "" H 3550 2200 50  0001 L CNN
 	1    3550 2200
@@
 F 0 "C7" H 4775 1900 50  0000 L CNN
 F 1 "C" H 4775 1700 50  0000 L CNN
-F 2 "Capacitors_SMD:C_0805_HandSoldering" H 4788 1650 50  0001 C CNN
+F 2 "drawdio:Resistor_SMD+THT" H 4788 1650 50  0001 C CNN
 F 3 "" H 4750 1800 50  0001 C CNN
 	1    4750 1800
@@
 F 0 "C8" H 4275 1250 50  0000 L CNN
 F 1 "C" H 4275 1050 50  0000 L CNN
-F 2 "Capacitors_SMD:C_0805_HandSoldering" H 4288 1000 50  0001 C CNN
+F 2 "drawdio:Resistor_SMD+THT" H 4288 1000 50  0001 C CNN
 F 3 "" H 4250 1150 50  0001 C CNN
 	1    4250 1150
@@
 F 0 "C10" H 6775 3300 50  0000 L CNN
 F 1 "C" H 6775 3100 50  0000 L CNN
-F 2 "Capacitors_SMD:C_0805_HandSoldering" H 6788 3050 50  0001 C CNN
+F 2 "drawdio:Resistor_SMD+THT" H 6788 3050 50  0001 C CNN
 F 3 "" H 6750 3200 50  0001 C CNN
 	1    6750 3200
@@
 F 0 "SW1" H 7025 4400 50  0000 C CNN
 F 1 "SW_TPDT" H 7500 4400 50  0000 C CNN
-F 2 "def-footprints:Switches_Stomp_Switch_3PDT" H 7200 4200 50  0001 C CNN
+F 2 "Wire_Pads:SolderWirePad_2x_1-5mmDrill" H 7200 4200 50  0001 C CNN
 F 3 "" H 7200 4200 50  0001 C CNN
 	1    7200 4200
@@
 F 0 "JP1" H 9850 4300 50  0000 C CNN
 F 1 "TB" H 9850 4070 50  0000 C CNN
-F 2 "" H 9850 4150 50  0001 C CNN
+F 2 "def-footprints:Miscellaneous_Solder_Jumper" H 9850 4150 50  0001 C CNN
 F 3 "" H 9850 4150 50  0001 C CNN
 	1    9850 4150
@@
 F 0 "JP20" H 9850 4650 50  0000 C CNN
 F 1 "PSEUDO" H 9850 4420 50  0000 C CNN
-F 2 "" H 9850 4500 50  0001 C CNN
+F 2 "def-footprints:Miscellaneous_Solder_Jumper" H 9850 4500 50  0001 C CNN
 F 3 "" H 9850 4500 50  0001 C CNN
 	1    9850 4500
@@
 F 0 "JP21" H 9850 5000 50  0000 C CNN
 F 1 "PSEUDO" H 9850 4770 50  0000 C CNN
-F 2 "" H 9850 4850 50  0001 C CNN
+F 2 "def-footprints:Miscellaneous_Solder_Jumper" H 9850 4850 50  0001 C CNN
 F 3 "" H 9850 4850 50  0001 C CNN
 	1    9850 4850
@@
 F 0 "Q2" H 9700 2725 50  0000 L CNN
 F 1 "2SC1815" H 9700 2650 50  0000 L CNN
-F 2 "TO_SOT_Packages_SMD:SOT-323_SC-70_Handsoldering" H 9700 2575 50  0001 L CIN
+F 2 "drawdio:TO-92_SOT23_JorFru_compact" H 9700 2575 50  0001 L CIN
 F 3 "" H 9500 2650 50  0001 L CNN
 	1    9500 2650
