File: KiCad/icescreamer.sch (KiCad schematic (older format))
At the start: 84 parts, among them J1 Audio-Jack-3_3Switches, J2 Audio-Jack-3_3Switches, Q1 2SC1815, Q2 2SC1815, Q20 2SC1815, Q21 2SC1815, Q22 2SC1815, Q23 Q_NJFET_SGD, Q24 Q_NJFET_SGD, SW1 SW_TPDT, SW20 SW_Push, U1 NE5532

Commit message: Añadidos archivos de huellas
DIP8+SOIC8 importado de Drawdio
3PDT tomado de def-footprints
Parts:
- BT1: footprint Wire_Pads:SolderWirePad_2x_1-2mmDrill -> Socket_Strips:Socket_Strip_Straight_1x02_Pitch2.54mm
- SW1: footprint Wire_Pads:SolderWirePad_2x_1-5mmDrill -> footprints:IceStomp_Switch_3PDT
- SW20: footprint def-footprints:Switches_Push_Switch_THD -> Socket_Strips:Socket_Strip_Straight_1x02_Pitch2.54mm
- U1: footprint (none) -> footprints:DIP8+SOIC8_2
Changed lines of the file:
@@
 F 0 "U1" H 4850 2500 50  0000 L CNN
 F 1 "NE5532" H 4850 2100 50  0000 L CNN
-F 2 "" H 4850 2300 50  0001 C CNN
+F 2 "footprints:DIP8+SOIC8_2" H 4850 2300 50  0001 C CNN
 F 3 "" H 4850 2300 50  0001 C CNN
 	1    4850 2300
@@
 F 0 "SW20" H 1150 6700 50  0000 L CNN
 F 1 "SW_Push" H 1100 6540 50  0000 C CNN
-F 2 "def-footprints:Switches_Push_Switch_THD" H 1100 6800 50  0001 C CNN
+F 2 "Socket_Strips:Socket_Strip_Straight_1x02_Pitch2.54mm" H 1100 6800 50  0001 C CNN
 F 3 "" H 1100 6800 50  0001 C CNN
 	1    1100 6600
@@
 F 0 "BT1" H 1100 1100 50  0000 L CNN
 F 1 "Battery_Cell" V 850 1000 50  0000 L CNN
-F 2 "Wire_Pads:SolderWirePad_2x_1-2mmDrill" V 1050 1210 50  0001 C CNN
+F 2 "Socket_Strips:Socket_Strip_Straight_1x02_Pitch2.54mm" V 1050 1210 50  0001 C CNN
 F 3 "" V 1050 1210 50  0001 C CNN
 	1    1050 1150
@@
 F 0 "SW1" H 7025 4400 50  0000 C CNN
 F 1 "SW_TPDT" H 7500 4400 50  0000 C CNN
-F 2 "Wire_Pads:SolderWirePad_2x_1-5mmDrill" H 7200 4200 50  0001 C CNN
+F 2 "footprints:IceStomp_Switch_3PDT" H 7200 4200 50  0001 C CNN
 F 3 "" H 7200 4200 50  0001 C CNN
 	1    7200 4200
@@
 F 0 "U1" H 6950 2600 50  0000 L CNN
 F 1 "NE5532" H 6950 2200 50  0000 L CNN
-F 2 "" H 6950 2400 50  0001 C CNN
+F 2 "footprints:DIP8+SOIC8_2" H 6950 2400 50  0001 C CNN
 F 3 "" H 6950 2400 50  0001 C CNN
 	2    6950 2400

Commit message: JorFru approved
Parts:
- added J3: Barrel_Jack_Switch, Connector_PinHeader_2.54mm:PinHeader_1x03_P2.54mm_Vertical, symbol Connector:Barrel_Jack_Switch
- BT1: footprint Socket_Strips:Socket_Strip_Straight_1x02_Pitch2.54mm -> drawdio:1x02_P2.54mm_Hole; symbol Battery_Cell -> icescreamer-rescue:Battery_Cell
- C1, C2: footprint Capacitors_THT:CP_Radial_D6.3mm_P2.50mm -> Capacitor_THT:CP_Radial_D6.3mm_P2.50mm; symbol CP -> icescreamer-rescue:CP
- C10, C7, C8: footprint drawdio:Resistor_SMD+THT -> Capacitor_THT:C_Rect_L7.0mm_W3.5mm_P2.50mm_P5.00mm; symbol C -> icescreamer-rescue:C
- C11, C12, C13, C20, C21, C22, C23, C24, C25, C26, C27, C6, C9: footprint Capacitors_SMD:C_0805_HandSoldering -> Capacitor_SMD:C_0805_2012Metric_Pad1.15x1.40mm_HandSolder; symbol C -> icescreamer-rescue:C
- C3, C4: footprint Capacitors_THT:C_Rect_L7.0mm_W3.5mm_P2.50mm_P5.00mm -> Capacitor_SMD:C_0805_2012Metric_Pad1.15x1.40mm_HandSolder; symbol C -> icescreamer-rescue:C
- C5: footprint drawdio:Resistor_SMD+THT -> Capacitor_SMD:C_0805_2012Metric_Pad1.15x1.40mm_HandSolder; symbol C -> icescreamer-rescue:C
- D1: footprint Capacitors_SMD:C_0805_HandSoldering -> Diode_THT:D_DO-41_SOD81_P7.62mm_Horizontal; symbol D -> icescreamer-rescue:D
- D2, D3: footprint Diodes_SMD:D_SOD-323_HandSoldering -> Diode_SMD:D_MELF-RM10_Universal_Handsoldering; symbol D -> icescreamer-rescue:D
- D20, D21, D22: footprint Diodes_SMD:D_SOD-323_HandSoldering -> Diode_SMD:D_0805_2012Metric_Pad1.15x1.40mm_HandSolder; symbol D -> icescreamer-rescue:D
- D23: footprint Diodes_SMD:D_SOD-323_HandSoldering -> Diode_SMD:D_MiniMELF_Handsoldering; symbol D_Zener -> icescreamer-rescue:D_Zener
- D4: footprint Pin_Headers:Pin_Header_Straight_1x02_Pitch2.54mm -> Connector_PinHeader_2.54mm:PinHeader_1x02_P2.54mm_Vertical; symbol LED -> icescreamer-rescue:LED
- J1, J2: symbol Audio-Jack-3_3Switches -> icescreamer-rescue:Audio-Jack-3_3Switches
- JP1, JP20, JP21: footprint def-footprints:Miscellaneous_Solder_Jumper -> Jumper:SolderJumper-2_P1.3mm_Open_RoundedPad1.0x1.5mm; symbol Jumper -> icescreamer-rescue:Jumper
- POT1, POT2, POT3: footprint footprints:IcePOT -> Connector_PinHeader_2.54mm:PinHeader_1x03_P2.54mm_Vertical; symbol POT -> icescreamer-rescue:POT
- Q1, Q2: symbol 2SC1815 -> icescreamer-rescue:2SC1815
- Q20, Q21, Q22: footprint TO_SOT_Packages_SMD:SOT-323_SC-70_Handsoldering -> drawdio:TO-92_SOT23_JorFru_compact; symbol 2SC1815 -> icescreamer-rescue:2SC1815
- Q23, Q24: footprint TO_SOT_Packages_SMD:SOT-323_SC-70_Handsoldering -> drawdio:TO-92_SOT23_JorFru_compact; symbol Q_NJFET_SGD -> icescreamer-rescue:Q_NJFET_SGD
- R1, R10, R11, R12, R13, R14, R15, R16, R17, R18, R19, R2, R20, R21, R22, R23, R24, R25, R26, R27, R28, R29, R3, R30, R31, R32, R33, R34, R35, R36, R4, R5, R6, R7, R8, R9: footprint Resistors_SMD:R_0805_HandSoldering -> Resistor_SMD:R_0805_2012Metric_Pad1.15x1.40mm_HandSolder; symbol R -> icescreamer-rescue:R
- SW1: symbol SW_TPDT -> icescreamer-rescue:SW_TPDT
- SW20: footprint Socket_Strips:Socket_Strip_Straight_1x02_Pitch2.54mm -> drawdio:1x02_P2.54mm_Hole; symbol SW_Push -> icescreamer-rescue:SW_Push
- U1: symbol NE5532 -> icescreamer-rescue:NE5532
Connections:
- net +VDC: now also U1.8 (V+), J3.2; no longer BT1.1 (+)
- net -VDC: now also U1.4 (V-)
- net BATT-: now also J3.1
- net at C6.1, R6.1: now also U1.3 (+); no longer U1.2 (-)
- net at C7.2, C8.1, D2.2 (A)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: now also U1.2 (-); no longer U1.3 (+)
- new net: BT1.1 (+), J3.3
Other:
- moved on the sheet: BT1, C1, C2, C3, C4, D1, R1, R2

Commit message: V0.3 ready
Parts:
- added C14, C15, C16, C17, C18: C, Capacitor_SMD:C_0805_2012Metric_Pad1.15x1.40mm_HandSolder, symbol icescreamer-rescue:C
- D4: footprint Connector_PinHeader_2.54mm:PinHeader_1x02_P2.54mm_Vertical -> Connector_PinHeader_2.00mm:PinHeader_1x02_P2.00mm_Vertical
Connections:
- net +VDC: now also C16.1
- net -VDC: now also C14.2, C15.2, C16.2, C17.2, C18.2
- net GNDREF: now also C14.1, C15.1, C17.1, C18.1
Other:
- moved on the sheet: C2, D1
Changed lines of the file:
@@
 F 0 "D4" H 7200 5900 50  0000 C CNN
 F 1 "LED" H 7200 5700 50  0000 C CNN
-F 2 "Connector_PinHeader_2.54mm:PinHeader_1x02_P2.54mm_Vertical" H 7200 5800 50  0001 C CNN
+F 2 "Connector_PinHeader_2.00mm:PinHeader_1x02_P2.00mm_Vertical" H 7200 5800 50  0001 C CNN
 F 3 "" H 7200 5800 50  0001 C CNN
 	1    7200 5800
@@
 L icescreamer-rescue:D D1
 U 1 1 5A2F0B86
-P 8700 1200
-F 0 "D1" H 8700 1300 50  0000 C CNN
-F 1 "D" H 8700 1100 50  0000 C CNN
-F 2 "Diode_THT:D_DO-41_SOD81_P7.62mm_Horizontal" H 8700 1200 50  0001 C CNN
-F 3 "" H 8700 1200 50  0001 C CNN
-	1    8700 1200
+P 8600 1200
+F 0 "D1" H 8350 1200 50  0000 C CNN
+F 1 "D" H 8700 1200 50  0000 C CNN
+F 2 "Diode_THT:D_DO-41_SOD81_P7.62mm_Horizontal" H 8600 1200 50  0001 C CNN
+F 3 "" H 8600 1200 50  0001 C CNN
+	1    8600 1200
 	0    1    1    0
 $EndComp
@@
 U 1 1 5A2F0C57
 P 9000 1200
-F 0 "C1" H 9025 1300 50  0000 L CNN
+F 0 "C1" H 9050 1300 50  0000 L CNN
 F 1 "CP" H 9025 1100 50  0000 L CNN
 F 2 "Capacitor_THT:CP_Radial_D6.3mm_P2.50mm" H 9038 1050 50  0001 C CNN
@@
 L icescreamer-rescue:CP C2
 U 1 1 5A2F1049
-P 9900 1350
-F 0 "C2" H 9925 1450 50  0000 L CNN
-F 1 "CP" H 9925 1250 50  0000 L CNN
-F 2 "Capacitor_THT:CP_Radial_D6.3mm_P2.50mm" H 9938 1200 50  0001 C CNN
-F 3 "" H 9900 1350 50  0001 C CNN
-	1    9900 1350
+P 9850 1350
+F 0 "C2" H 9875 1450 50  0000 L CNN
+F 1 "CP" H 9875 1250 50  0000 L CNN
+F 2 "Capacitor_THT:CP_Radial_D6.3mm_P2.50mm" H 9888 1200 50  0001 C CNN
+F 3 "" H 9850 1350 50  0001 C CNN
+	1    9850 1350
 	1    0    0    -1
 $EndComp
@@
 $EndComp
 $Comp
-L icescreamer-rescue:GNDREF #PWR034
-U 1 1 5A342630
-P 10200 1200
-F 0 "#PWR034" H 10200 950 50  0001 C CNN
-F 1 "GNDREF" H 10200 1050 50  0000 C CNN
-F 2 "" H 10200 1200 50  0001 C CNN
-F 3 "" H 10200 1200 50  0001 C CNN
-	1    10200 1200
-	1    0    0    -1
-$EndComp
-$Comp
 L icescreamer-rescue:-VDC #PWR035
 U 1 1 5A3426E7
@@
 L icescreamer-rescue:PWR_FLAG #FLG037
 U 1 1 5A342963
-P 10200 1200
-F 0 "#FLG037" H 10200 1275 50  0001 C CNN
-F 1 "PWR_FLAG" H 10200 1350 50  0000 C CNN
-F 2 "" H 10200 1200 50  0001 C CNN
-F 3 "" H 10200 1200 50  0001 C CNN
-	1    10200 1200
+P 10500 900
+F 0 "#FLG037" H 10500 975 50  0001 C CNN
+F 1 "PWR_FLAG" H 10500 1050 50  0000 C CNN
+F 2 "" H 10500 900 50  0001 C CNN
+F 3 "" H 10500 900 50  0001 C CNN
+	1    10500 900
 	1    0    0    -1
 $EndComp
@@
 	-1   0    0    1
 $EndComp
-Connection ~ 9900 1200
 Connection ~ 8350 2650
 Wire Wire Line
@@
 	9000 1500 9300 1500
 Wire Wire Line
-	8700 1350 9000 1350
-Wire Wire Line
 	9000 900  9300 900
 Wire Wire Line
 	9000 1050 9000 900
-Connection ~ 8700 1050
 Wire Wire Line
 	7200 5950 7200 6050
@@
 	8950 6050 9000 6050
 Wire Wire Line
-	9900 1200 10200 1200
-Wire Wire Line
 	8350 2650 8650 2650
 Wire Wire Line
@@
 	9300 900  9600 900
 Wire Wire Line
-	9600 1200 9900 1200
-Wire Wire Line
-	9600 1500 9900 1500
+	9600 1200 9850 1200
+Wire Wire Line
+	9600 1500 9850 1500
 Wire Wire Line
 	9300 1500 9600 1500
-Wire Wire Line
-	8700 1050 9000 1050
 $Comp
 L icescreamer-rescue:NE5532 U1
@@
 Connection ~ 9300 1200
 Connection ~ 9600 900
-Connection ~ 10200 1200
 Wire Wire Line
 	8000 1400 8000 1600
@@
 	8000 1200 8000 1050
 Wire Wire Line
-	8000 1050 8700 1050
+	8000 1050 8600 1050
 $Comp
 L icescreamer-rescue:+VDC #PWR0102
@@
 PSEUDO_IN_1
 Connection ~ 7250 2400
+$Comp
+L icescreamer-rescue:C C14
+U 1 1 5E4A17DA
+P 10100 1350
+F 0 "C14" H 10125 1450 50  0000 L CNN
+F 1 "C" H 10125 1250 50  0000 L CNN
+F 2 "Capacitor_SMD:C_0805_2012Metric_Pad1.15x1.40mm_HandSolder" H 10138 1200 50  0001 C CNN
+F 3 "" H 10100 1350 50  0001 C CNN
+	1    10100 1350
+	1    0    0    -1
+$EndComp
+$Comp
+L icescreamer-rescue:C C15
+U 1 1 5E4A1E61
+P 10300 1350
+F 0 "C15" H 10325 1450 50  0000 L CNN
+F 1 "C" H 10325 1250 50  0000 L CNN
+F 2 "Capacitor_SMD:C_0805_2012Metric_Pad1.15x1.40mm_HandSolder" H 10338 1200 50  0001 C CNN
+F 3 "" H 10300 1350 50  0001 C CNN
+	1    10300 1350
+	1    0    0    -1
+$EndComp
+$Comp
+L icescreamer-rescue:C C16
+U 1 1 5E4A2346
+P 8800 1200
+F 0 "C16" H 8750 1450 50  0000 L CNN
+F 1 "C" H 8825 1100 50  0000 L CNN
+F 2 "Capacitor_SMD:C_0805_2012Metric_Pad1.15x1.40mm_HandSolder" H 8838 1050 50  0001 C CNN
+F 3 "" H 8800 1200 50  0001 C CNN
+	1    8800 1200
+	1    0    0    -1
+$EndComp
+$Comp
+L icescreamer-rescue:GNDREF #PWR034
+U 1 1 5A342630
+P 10500 900
+F 0 "#PWR034" H 10500 650 50  0001 C CNN
+F 1 "GNDREF" H 10500 750 50  0000 C CNN
+F 2 "" H 10500 900 50  0001 C CNN
+F 3 "" H 10500 900 50  0001 C CNN
+	1    10500 900
+	1    0    0    -1
+$EndComp
+$Comp
+L icescreamer-rescue:C C17
+U 1 1 5E4CF043
+P 10500 1350
+F 0 "C17" H 10525 1450 50  0000 L CNN
+F 1 "C" H 10525 1250 50  0000 L CNN
+F 2 "Capacitor_SMD:C_0805_2012Metric_Pad1.15x1.40mm_HandSolder" H 10538 1200 50  0001 C CNN
+F 3 "" H 10500 1350 50  0001 C CNN
+	1    10500 1350
+	1    0    0    -1
+$EndComp
+$Comp
+L icescreamer-rescue:C C18
+U 1 1 5E4CF526
+P 10700 1350
+F 0 "C18" H 10725 1450 50  0000 L CNN
+F 1 "C" H 10725 1250 50  0000 L CNN
+F 2 "Capacitor_SMD:C_0805_2012Metric_Pad1.15x1.40mm_HandSolder" H 10738 1200 50  0001 C CNN
+F 3 "" H 10700 1350 50  0001 C CNN
+	1    10700 1350
+	1    0    0    -1
+$EndComp
+Wire Wire Line
+	10100 1500 10300 1500
+Connection ~ 10100 1500
+Connection ~ 10300 1500
+Wire Wire Line
+	10100 1200 10300 1200
+Connection ~ 10100 1200
+Connection ~ 10300 1200
+Wire Wire Line
+	10700 900  10500 900
+Connection ~ 10500 900
+Connection ~ 9850 1200
+Connection ~ 9850 1500
+Wire Wire Line
+	9850 1500 10100 1500
+Wire Wire Line
+	9850 1200 10100 1200
+Wire Wire Line
+	10300 1200 10500 1200
+Wire Wire Line
+	10300 1500 10500 1500
+Connection ~ 10500 1200
+Wire Wire Line
+	10500 1200 10700 1200
+Connection ~ 10500 1500
+Wire Wire Line
+	10500 1500 10700 1500
+Wire Wire Line
+	10700 1200 10700 900
+Connection ~ 10700 1200
+Connection ~ 8600 1050
+Wire Wire Line
+	8600 1050 8800 1050
+Wire Wire Line
+	8600 1350 8800 1350
+Connection ~ 8800 1050
+Wire Wire Line
+	8800 1050 9000 1050
+Connection ~ 8800 1350
+Wire Wire Line
+	8800 1350 9000 1350
 $EndSCHEMATC
