File: KiCad/icescreamer.sch (KiCad schematic (older format))
At the start: 90 parts, among them J1 Audio-Jack-3_3Switches, J2 Audio-Jack-3_3Switches, J3 Barrel_Jack_Switch, Q1 2SC1815, Q2 2SC1815, Q20 2SC1815, Q21 2SC1815, Q22 2SC1815, Q23 Q_NJFET_SGD, Q24 Q_NJFET_SGD, SW1 SW_TPDT, SW20 SW_Push, U1 NE5532

Commit message: V0.3 release
Parts:
- removed Q1, Q2, Q20, Q21, Q22: 2SC1815, drawdio:TO-92_SOT23_JorFru_compact, symbol icescreamer-rescue:2SC1815
- added Q1, Q2, Q20, Q21, Q22: BC547, IceScreamer:TO-92_SOT23_JorFru_compact, symbol Transistor_BJT:BC547
Connections:
- net +VDC: now also Q1.1 (C), Q2.1 (C)
- net PSEUDO_IN_1: now also Q1.3 (E)
- net at R3.1, R4.1: now also Q1.2 (B)
- net at C12.1, R14.1: now also Q2.2 (B)
- net at C23.2, R22.2, R23.2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: now also Q20.1 (C)
- net at D22.2 (A): now also Q20.3 (E), Q21.3 (E), Q22.3 (E)
- net at C24.2, C25.2, R29.1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: now also Q20.2 (B)
- net at C24.1, R29.2, R32.2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: now also Q21.1 (C)
- net at C23.1, C26.2, R28.2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: now also Q21.2 (B)
- net at R33.2: now also Q22.2 (B)
- net at D23.2 (A): now also Q22.1 (C)
- net at R15.1, R16.2: now also Q2.3 (E)
Changed lines of the file:
@@
-$EndComp
-$Comp
-L icescreamer-rescue:2SC1815 Q1
-U 1 1 5A2D758C
-P 3550 2200
-F 0 "Q1" H 3750 2275 50  0000 L CNN
-F 1 "2SC1815" H 3750 2200 50  0000 L CNN
-F 2 "drawdio:TO-92_SOT23_JorFru_compact" H 3750 2125 50  0001 L CIN
-F 3 "" H 3550 2200 50  0001 L CNN
-	1    3550 2200
-	1    0    0    -1
 $EndComp
 $Comp
@@
 $EndComp
 $Comp
-L icescreamer-rescue:2SC1815 Q20
-U 1 1 5A2E7B18
-P 2600 5400
-F 0 "Q20" H 2800 5475 50  0000 L CNN
-F 1 "2SC1815" H 2800 5400 50  0000 L CNN
-F 2 "drawdio:TO-92_SOT23_JorFru_compact" H 2800 5325 50  0001 L CIN
-F 3 "" H 2600 5400 50  0001 L CNN
-	1    2600 5400
-	-1   0    0    -1
-$EndComp
-$Comp
 L icescreamer-rescue:R R30
 U 1 1 5A2E7BF1
@@
 $EndComp
 $Comp
-L icescreamer-rescue:2SC1815 Q21
-U 1 1 5A2E84FA
-P 4250 5400
-F 0 "Q21" H 4450 5475 50  0000 L CNN
-F 1 "2SC1815" H 4450 5400 50  0000 L CNN
-F 2 "drawdio:TO-92_SOT23_JorFru_compact" H 4450 5325 50  0001 L CIN
-F 3 "" H 4250 5400 50  0001 L CNN
-	1    4250 5400
-	1    0    0    -1
-$EndComp
-$Comp
 L icescreamer-rescue:R R33
 U 1 1 5A2E8627
@@
 	1    5300 6050
 	0    1    1    0
-$EndComp
-$Comp
-L icescreamer-rescue:2SC1815 Q22
-U 1 1 5A2E9060
-P 5200 6450
-F 0 "Q22" H 5400 6525 50  0000 L CNN
-F 1 "2SC1815" H 5400 6450 50  0000 L CNN
-F 2 "drawdio:TO-92_SOT23_JorFru_compact" H 5400 6375 50  0001 L CIN
-F 3 "" H 5200 6450 50  0001 L CNN
-	1    5200 6450
-	1    0    0    -1
 $EndComp
 $Comp
@@
 $EndComp
 $Comp
-L icescreamer-rescue:2SC1815 Q2
-U 1 1 5A317C1E
-P 9500 2650
-F 0 "Q2" H 9700 2725 50  0000 L CNN
-F 1 "2SC1815" H 9700 2650 50  0000 L CNN
-F 2 "drawdio:TO-92_SOT23_JorFru_compact" H 9700 2575 50  0001 L CIN
-F 3 "" H 9500 2650 50  0001 L CNN
-	1    9500 2650
-	1    0    0    -1
-$EndComp
-$Comp
 L icescreamer-rescue:R R15
 U 1 1 5A31884E
@@
 	5000 6450 4700 6450
 Connection ~ 4700 5200
-Connection ~ 4350 5200
-Wire Wire Line
-	4050 5200 4350 5200
 Wire Wire Line
 	4050 5000 4050 5200
@@
 Wire Wire Line
 	2800 5200 2800 5000
-Connection ~ 2500 5200
 Connection ~ 1750 5200
 Wire Wire Line
@@
 Wire Wire Line
 	3800 2400 3800 2450
-Connection ~ 3650 2400
-Wire Wire Line
-	3500 2400 3650 2400
 Wire Wire Line
 	3500 2450 3500 2400
@@
 	4700 5200 4850 5200
 Wire Wire Line
-	4350 5200 4700 5200
-Wire Wire Line
 	4350 6650 5300 6650
 Wire Wire Line
@@
 	2950 5400 2800 5400
 Wire Wire Line
-	2500 5200 2800 5200
-Wire Wire Line
 	1750 5200 1900 5200
 Wire Wire Line
@@
 Wire Wire Line
 	3800 2400 4000 2400
-Wire Wire Line
-	3650 2400 3800 2400
 Wire Wire Line
 	3200 2200 3350 2200
@@
 PSEUDO_IN_1
 Wire Wire Line
-	2350 5200 2500 5200
-Wire Wire Line
 	2200 5200 2350 5200
 Connection ~ 2350 5200
@@
 Wire Wire Line
 	8800 1350 9000 1350
+$Comp
+L Transistor_BJT:BC547 Q1
+U 1 1 5E39C402
+P 3550 2200
+F 0 "Q1" H 3741 2246 50  0000 L CNN
+F 1 "BC547" H 3741 2155 50  0000 L CNN
+F 2 "IceScreamer:TO-92_SOT23_JorFru_compact" H 3750 2125 50  0001 L CIN
+F 3 "http://www.fairchildsemi.com/ds/BC/BC547.pdf" H 3550 2200 50  0001 L CNN
+	1    3550 2200
+	1    0    0    -1
+$EndComp
+Wire Wire Line
+	3500 2400 3650 2400
+Connection ~ 3650 2400
+Wire Wire Line
+	3650 2400 3800 2400
+$Comp
+L Transistor_BJT:BC547 Q2
+U 1 1 5E3ADD8B
+P 9500 2650
+F 0 "Q2" H 9691 2696 50  0000 L CNN
+F 1 "BC547" H 9691 2605 50  0000 L CNN
+F 2 "IceScreamer:TO-92_SOT23_JorFru_compact" H 9700 2575 50  0001 L CIN
+F 3 "http://www.fairchildsemi.com/ds/BC/BC547.pdf" H 9500 2650 50  0001 L CNN
+	1    9500 2650
+	1    0    0    -1
+$EndComp
+Connection ~ 9600 2850
+$Comp
+L Transistor_BJT:BC547 Q22
+U 1 1 5E3B2793
+P 5200 6450
+F 0 "Q22" H 5391 6496 50  0000 L CNN
+F 1 "BC547" H 5391 6405 50  0000 L CNN
+F 2 "IceScreamer:TO-92_SOT23_JorFru_compact" H 5400 6375 50  0001 L CIN
+F 3 "http://www.fairchildsemi.com/ds/BC/BC547.pdf" H 5200 6450 50  0001 L CNN
+	1    5200 6450
+	1    0    0    -1
+$EndComp
+Connection ~ 5300 6650
+$Comp
+L Transistor_BJT:BC547 Q21
+U 1 1 5E3BA1E3
+P 4250 5400
+F 0 "Q21" H 4441 5446 50  0000 L CNN
+F 1 "BC547" H 4441 5355 50  0000 L CNN
+F 2 "IceScreamer:TO-92_SOT23_JorFru_compact" H 4450 5325 50  0001 L CIN
+F 3 "http://www.fairchildsemi.com/ds/BC/BC547.pdf" H 4250 5400 50  0001 L CNN
+	1    4250 5400
+	1    0    0    -1
+$EndComp
+Wire Wire Line
+	4050 5200 4350 5200
+Connection ~ 4350 5200
+Wire Wire Line
+	4350 5200 4700 5200
+$Comp
+L Transistor_BJT:BC547 Q20
+U 1 1 5E3C4791
+P 2600 5400
+F 0 "Q20" H 2791 5446 50  0000 L CNN
+F 1 "BC547" H 2791 5355 50  0000 L CNN
+F 2 "IceScreamer:TO-92_SOT23_JorFru_compact" H 2800 5325 50  0001 L CIN
+F 3 "http://www.fairchildsemi.com/ds/BC/BC547.pdf" H 2600 5400 50  0001 L CNN
+	1    2600 5400
+	-1   0    0    -1
+$EndComp
+Wire Wire Line
+	2350 5200 2500 5200
+Connection ~ 2500 5200
+Wire Wire Line
+	2500 5200 2800 5200
 $EndSCHEMATC
